File: STMF4_BreadBoardBreakout/STMF4_BreadBoardBreakout.sch (KiCad schematic (older format))
At the start: 48 parts, among them IC1 SGM2019-ADJYN5G-TR, J1 USART1, J10 PORT D, J11 PORT E, J2 USB_B_Micro, J3 USART2, J4 SWD, J5 I2C3, J6 SPI1, J7 PORT A, J8 PORT B, J9 PORT C, U1 STM32F446VETx, Y1 Crystal

Commit message: rough component placement, change to smd
Parts:
- removed H1, H2, H3, H4: MountingHole_Pad, MountingHole:MountingHole_3.5mm_Pad, symbol Mechanical:MountingHole_Pad
- added C18, C19: 10uF, Capacitor_SMD:C_0603_1608Metric, symbol STMF4_BreadBoardBreakout-rescue:C_Small-Device
- added J12: DCMI SPI CAM, Connector_PinSocket_2.54mm:PinSocket_2x09_P2.54mm_Vertical_SMD, symbol Connector_Generic:Conn_02x09_Odd_Even
- added R10, R12: 10k, Resistor_SMD:R_0603_1608Metric_Pad1.05x0.95mm_HandSolder, symbol STMF4_BreadBoardBreakout-rescue:R_Small-Device
- added R11, R13: 1k, Resistor_SMD:R_0603_1608Metric_Pad1.05x0.95mm_HandSolder, symbol STMF4_BreadBoardBreakout-rescue:R_Small-Device
- added SW1: BTN_NRST, Button_Switch_SMD:SW_SPST_SKQG_WithStem, symbol Switch:SW_Push
- added SW2: BTN_UTIL1, Button_Switch_SMD:SW_SPST_SKQG_WithStem, symbol Switch:SW_Push
- C1, C10, C11, C12, C13, C14, C15, C16, C17, C2, C3, C4, C5, C6, C7, C8, C9: footprint Capacitor_SMD:C_0603_1608Metric_Pad1.05x0.95mm_HandSolder -> Capacitor_SMD:C_0603_1608Metric; symbol Device:C_Small -> STMF4_BreadBoardBreakout-rescue:C_Small-Device
- D1: footprint Diode_THT:D_DO-15_P10.16mm_Horizontal -> Diode_SMD:D_0603_1608Metric; symbol Device:D_Schottky -> STMF4_BreadBoardBreakout-rescue:D_Schottky-Device
- D2, D3: footprint LED_THT:LED_D5.0mm -> Diode_SMD:D_0603_1608Metric; symbol Device:LED_Small -> STMF4_BreadBoardBreakout-rescue:LED_Small-Device
- F1: footprint (none) -> Fuse:Fuse_1206_3216Metric; symbol Device:Fuse -> STMF4_BreadBoardBreakout-rescue:Fuse-Device
- IC1: footprint Package_TO_SOT_SMD:SOT-23-5_HandSoldering -> Package_TO_SOT_SMD:SOT-23-5; symbol SGM2019:SGM2019-ADJYN5G-TR -> STMF4_BreadBoardBreakout-rescue:SGM2019-ADJYN5G-TR-SGM2019
- J1, J3: symbol Connector:Conn_01x03_Male -> STMF4_BreadBoardBreakout-rescue:Conn_01x03_Male-Connector
- J10, J7, J8, J9: symbol Connector:Conn_01x16_Male -> STMF4_BreadBoardBreakout-rescue:Conn_01x16_Male-Connector
- J11: footprint Connector_PinHeader_1.27mm:PinHeader_1x16_P1.27mm_Vertical -> Connector_PinHeader_2.54mm:PinHeader_1x16_P2.54mm_Vertical; symbol Connector:Conn_01x16_Male -> STMF4_BreadBoardBreakout-rescue:Conn_01x16_Male-Connector
- J2: footprint Connector_USB:USB_Micro-B_Amphenol_10103594-0001LF_Horizontal -> Connector_USB:USB_Micro-B_Wuerth_629105150521; symbol Connector:USB_B_Micro -> STMF4_BreadBoardBreakout-rescue:USB_B_Micro-Connector
- J4: symbol Connector:Conn_01x06_Female -> STMF4_BreadBoardBreakout-rescue:Conn_01x06_Female-Connector
- J5: symbol Connector:Conn_01x04_Male -> STMF4_BreadBoardBreakout-rescue:Conn_01x04_Male-Connector
- J6: symbol Connector:Conn_01x06_Male -> STMF4_BreadBoardBreakout-rescue:Conn_01x06_Male-Connector
- R1, R2, R3, R4, R5, R6, R7, R8, R9: symbol Device:R_Small -> STMF4_BreadBoardBreakout-rescue:R_Small-Device
- U1: symbol MCU_ST_STM32F4:STM32F446VETx -> STMF4_BreadBoardBreakout-rescue:STM32F446VETx-MCU_ST_STM32F4
- Y1: footprint Crystal:Crystal_DS15_D1.5mm_L5.0mm_Horizontal -> Crystal:Crystal_SMD_7050-4Pin_7.0x5.0mm; symbol Device:Crystal -> STMF4_BreadBoardBreakout-rescue:Crystal-Device
Connections:
- net +3.3VA: now also J12.1 (Pin_1), R10.2, R12.2
- net BOOT0: no longer R9.1
- net BOOT1: now also R9.1
- net GND: now also C18.2, C19.2, J12.2 (Pin_2), SW1.2, SW2.2
- net I2C3_SCL: now also J12.4 (Pin_4)
- net I2C3_SDA: now also J12.3 (Pin_3)
- new net: R11.1, SW1.1
- new net: R13.1, SW2.1
- new net: C18.1, R10.1, R11.2
- new net: C19.1, R12.1, R13.2
- new net D0: J12.15 (Pin_15)
- new net D1: J12.16 (Pin_16)
- new net D2: J12.13 (Pin_13)
- new net D3: J12.14 (Pin_14)
- new net D4: J12.11 (Pin_11)
- new net D5: J12.12 (Pin_12)
- new net D6: J12.9 (Pin_9)
- new net D7: J12.10 (Pin_10)
- new net HS: J12.5 (Pin_5)
- new net MCLK: J12.7 (Pin_7)
- new net PCLK: J12.8 (Pin_8)
- new net PWDN: J12.17 (Pin_17)
- new net RESET: J12.18 (Pin_18)
- new net VS: J12.6 (Pin_6)
Other:
- note added: "Buttons\nwith debouncing"
- note removed: "RESET + PUSHBUTTON"

Commit message: move connectors and mcu in sub schematic
Parts:
- removed J1: USART1, Connector_JST:JST_EH_S3B-EH_1x03_P2.50mm_Horizontal, symbol STMF4_BreadBoardBreakout-rescue:Conn_01x03_Male-Connector
- removed J10: PORT D, Connector_PinHeader_2.54mm:PinHeader_1x16_P2.54mm_Vertical, symbol STMF4_BreadBoardBreakout-rescue:Conn_01x16_Male-Connector
- removed J11: PORT E, Connector_PinHeader_2.54mm:PinHeader_1x16_P2.54mm_Vertical, symbol STMF4_BreadBoardBreakout-rescue:Conn_01x16_Male-Connector
- removed J12: DCMI SPI CAM, Connector_PinSocket_2.54mm:PinSocket_2x09_P2.54mm_Vertical_SMD, symbol Connector_Generic:Conn_02x09_Odd_Even
- removed J2: USB_B_Micro, Connector_USB:USB_Micro-B_Wuerth_629105150521, symbol STMF4_BreadBoardBreakout-rescue:USB_B_Micro-Connector
- removed J3: USART2, Connector_JST:JST_EH_S3B-EH_1x03_P2.50mm_Horizontal, symbol STMF4_BreadBoardBreakout-rescue:Conn_01x03_Male-Connector
- removed J4: SWD, Connector_PinSocket_2.54mm:PinSocket_1x06_P2.54mm_Vertical, symbol STMF4_BreadBoardBreakout-rescue:Conn_01x06_Female-Connector
- removed J5: I2C3, Connector_JST:JST_PH_S4B-PH-K_1x04_P2.00mm_Horizontal, symbol STMF4_BreadBoardBreakout-rescue:Conn_01x04_Male-Connector
- removed J6: SPI1, Connector_JST:JST_EH_S6B-EH_1x06_P2.50mm_Horizontal, symbol STMF4_BreadBoardBreakout-rescue:Conn_01x06_Male-Connector
- removed J7: PORT A, Connector_PinHeader_2.54mm:PinHeader_1x16_P2.54mm_Vertical, symbol STMF4_BreadBoardBreakout-rescue:Conn_01x16_Male-Connector
- removed J8: PORT B, Connector_PinHeader_2.54mm:PinHeader_1x16_P2.54mm_Vertical, symbol STMF4_BreadBoardBreakout-rescue:Conn_01x16_Male-Connector
- removed J9: PORT C, Connector_PinHeader_2.54mm:PinHeader_1x16_P2.54mm_Vertical, symbol STMF4_BreadBoardBreakout-rescue:Conn_01x16_Male-Connector
- removed U1: STM32F446VETx, Package_QFP:LQFP-100_14x14mm_P0.5mm, symbol STMF4_BreadBoardBreakout-rescue:STM32F446VETx-MCU_ST_STM32F4
- C1, C10, C11, C12, C13, C14, C15, C16, C17, C18, C19, C2, C3, C4, C5, C6, C7, C8, C9: symbol STMF4_BreadBoardBreakout-rescue:C_Small-Device -> STMF4_BreadBoardBreakout-rescue:C_Small-Device-STMF4_BreadBoardBreakout-rescue
- D1: symbol STMF4_BreadBoardBreakout-rescue:D_Schottky-Device -> STMF4_BreadBoardBreakout-rescue:D_Schottky-Device-STMF4_BreadBoardBreakout-rescue
- D2, D3: symbol STMF4_BreadBoardBreakout-rescue:LED_Small-Device -> STMF4_BreadBoardBreakout-rescue:LED_Small-Device-STMF4_BreadBoardBreakout-rescue
- F1: symbol STMF4_BreadBoardBreakout-rescue:Fuse-Device -> STMF4_BreadBoardBreakout-rescue:Fuse-Device-STMF4_BreadBoardBreakout-rescue
- IC1: symbol STMF4_BreadBoardBreakout-rescue:SGM2019-ADJYN5G-TR-SGM2019 -> STMF4_BreadBoardBreakout-rescue:SGM2019-ADJYN5G-TR-SGM2019-STMF4_BreadBoardBreakout-rescue
- R1, R10, R11, R12, R13, R2, R3, R4, R5, R6, R7, R8, R9: symbol STMF4_BreadBoardBreakout-rescue:R_Small-Device -> STMF4_BreadBoardBreakout-rescue:R_Small-Device-STMF4_BreadBoardBreakout-rescue
- Y1: symbol STMF4_BreadBoardBreakout-rescue:Crystal-Device -> STMF4_BreadBoardBreakout-rescue:Crystal-Device-STMF4_BreadBoardBreakout-rescue
Connections:
- no-connect marks 7 -> 0
Other:
- note added: "EXTRA PERIPHERAL SETUP"
- note added: "Microcontroller SETUP"
- note added: "POWER SUPPLY\n"
- note removed: "-> limit inrush current"
- note removed: "BreadBoard Connection\n"
- note removed: "Connectors\n"
- note removed: "DCMI for camera\n"
- note removed: "JLCPCB Impendence Calculator for Differnential lines"
- note removed: "Microcontroller"
- note removed: "SPI Reset?"
- note removed: "STM32 µC already matching impedence to usb DP, DM"
- note removed: "SWD - ST Link\n\n"
- note removed: "USB Connector\n"
- note removed: "USB host -side cap <= 10uF Micro USB \n\n"
- note removed: "match diff trace length, max time diff 1ps"
- note removed: "no pullups etc required (internal pull-up resistors , AN4879)\n"
- note removed: "possible esd protection: USBLC6-2SC6"
- note removed: "shield grounded to host, NC to PCB!\n"
- note removed: "testpoints\n"
- note removed: "todo check again\n\n"
- moved on the sheet: C1, C10, C11, C12, C13, C14, C15, C16, C17, C18, C19, C2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

Commit message: reduce size in pcb, fix second sheet, main routing finished
Parts:
- removed C11: 100nF, Capacitor_SMD:C_0603_1608Metric, symbol STMF4_BreadBoardBreakout-rescue:C_Small-Device-STMF4_BreadBoardBreakout-rescue
- removed C12: 1nF, Capacitor_SMD:C_0603_1608Metric, symbol STMF4_BreadBoardBreakout-rescue:C_Small-Device-STMF4_BreadBoardBreakout-rescue
- removed C17: 2.2uF, Capacitor_SMD:C_0603_1608Metric, symbol STMF4_BreadBoardBreakout-rescue:C_Small-Device-STMF4_BreadBoardBreakout-rescue
- renumbered C16 to C1, C1 to C11, C2 to C12, C3 to C13, C5 to C14, C6 to C15, C7 to C16, C8 to C17, C4 to C2, C15 to C3, C18 to C4, C19 to C6, C13 to C7, C9 to C8, C14 to C9, D3 to D2, D2 to D3, R6 to R1, R3 to R10, R4 to R11, R8 to R12, R5 to R13, R7 to R2, R9 to R3, R10 to R4, R11 to R5, R1 to R6, R2 to R7, R12 to R8, R13 to R9
Connections:
- net +3.3VA: no longer C10.1, C11.1, C12.1, C13.1, C14.1, C15.1, C16.1, C17.1, C8.1, D3.2 (A), IC1.5 (OUT), R11.1, R13.1, R4.2, R6.1, R8.2
- new net +3.3V: C10.1, C11.1, C12.1, C13.1, C14.1, C15.1, C16.1, C17.1, C8.1, D3.2 (A), IC1.5 (OUT), R11.1, R13.1, R4.2, R6.1, R8.2
Other:
- note added: "TODO: hf filter?\n"
- note added: "vCap2 missing`?"
- note removed: "ADC Supply\n"
- note removed: "hf filter\n"
- moved on the sheet: C11, C12, C13, C14, C15, C16, C17
